File: Melhorando-Heater.kicad_sch (KiCad schematic)
At the start: 0 parts

Commit message: :minidisc: finalizada placa problemática
Parts:
- added C1: 1n, Capacitor_SMD:C_0603_1608Metric, symbol Device:C_Small
- added C2: 100n, Capacitor_SMD:C_0603_1608Metric, symbol Device:C_Small
- added C3: 220uF 16V, Capacitor_SMD:CP_Elec_6.3x5.2, symbol Device:C_Polarized
- added D1: GREEN, LED_SMD:LED_0805_2012Metric, symbol Device:LED
- added D2, D3: RED, LED_SMD:LED_0805_2012Metric, symbol Device:LED
- added H1, H2, H3, H4: M3, MountingHole:MountingHole_3.2mm_M3, symbol Mechanical:MountingHole
- added J1: Conn_01x04, Connector_PinSocket_2.54mm:PinSocket_1x04_P2.54mm_Vertical, symbol Connector_Generic:Conn_01x04
- added J2: 1x03, TerminalBlock_Phoenix:TerminalBlock_Phoenix_MKDS-1,5-3-5.08_1x03_P5.08mm_Horizontal, symbol Connector:Screw_Terminal_01x03
- added J3: 1x04, TerminalBlock_Phoenix:TerminalBlock_Phoenix_MKDS-1,5-4-5.08_1x04_P5.08mm_Horizontal, symbol Connector:Screw_Terminal_01x04
- added Q1: BC817, Package_TO_SOT_SMD:SOT-23, symbol Transistor_BJT:BC817
- added R1: 47k, Resistor_SMD:R_0603_1608Metric, symbol Device:R_Small_US
- added R2, R3, R8: 10, Resistor_SMD:R_0603_1608Metric, symbol Device:R_Small_US
- added R4, R5, R6, R7: 470, Resistor_SMD:R_0603_1608Metric, symbol Device:R_Small_US
- added U1: MSP430FR2433IRGET, Package_DFN_QFN:VQFN-24-1EP_4x4mm_P0.5mm_EP2.45x2.45mm, symbol MSP430FR2433:MSP430FR2433IRGET
Connections:
- new net: D3.2 (A), R7.2
- new net: D2.2 (A), R6.2
- new net: Q1.1 (B), R4.2
- new net: D1.2 (A), R5.2
- new net 12V: C3.1, J2.1 (Pin_1), J3.1 (Pin_1)
- new net 3V3: C2.1, J1.1 (Pin_1), J2.2 (Pin_2), R1.1, U1.24 (DVCC)
- new net GND: C1.2, C2.2, C3.2, D1.1 (K), D2.1 (K), D3.1 (K), J1.4 (Pin_4), J2.3 (Pin_3), J3.4 (Pin_4), Q1.2 (E), U1.18 (DVSS), U1.23 (DVSS), U1.25 (PAD)
- new net LED_FAULT: R6.1, U1.16 (P2.5_UCA1RXD_UCA1SOMI)
- new net LED_HEAT: R7.1, U1.17 (P2.6_UCA1TXD_UCA1SIMO)
- new net LED_ON: R5.1, U1.15 (P2.4_UCA1CLK)
- new net MCU_DIO: R3.1, U1.1 (RST_NMI_SBWTDIO)
- new net MCU_RST: C1.1, R1.2, R2.1, U1.2 (TEST_SBWTCK)
- new net M_HEATER: R4.1, U1.5 (P1.6_UCA0CLK_TA1CLK_TDI_TCLK_A6)
- new net P_HEATER: J3.3 (Pin_3), Q1.3 (C)
- new net P_SENSOR: J3.2 (Pin_2), R8.2
- new net SBW_DIO: J1.3 (Pin_3), R3.2
- new net SBW_RST: J1.2 (Pin_2), R2.2
- new net S_SENSOR: R8.1, U1.8 (P1.1_UCB0CLK_TA0.1_A1)
Other:
- note added: "12V"
- note added: "3V3"
- note added: "GND"
- note added: "HEATER"
- note added: "SENSOR"

Commit message: :minidisc: delivered finished board
Connections:
- net 12V: now also J3.4 (Pin_4); no longer J3.1 (Pin_1)
- net GND: now also J3.1 (Pin_1); no longer J3.4 (Pin_4)
- net P_HEATER: now also J3.2 (Pin_2); no longer J3.3 (Pin_3)
- net P_SENSOR: now also J3.3 (Pin_3); no longer J3.2 (Pin_2)
Changed lines of the file:
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@@
 	(symbol
 		(lib_id "Connector:Screw_Terminal_01x04")
-		(at 246.38 69.85 0)
+		(at 246.38 72.39 0)
+		(mirror x)
 		(unit 1)
 		(exclude_from_sim no)
@@
 		(dnp no)
 		(property "Reference" "J3"
-			(at 245.364 64.516 0)
+			(at 245.364 64.77 0)
 			(effects
 				(font
@@
 		)
 		(property "Value" "1x04"
-			(at 244.094 77.47 0)
+			(at 244.348 77.724 0)
 			(effects
 				(font
@@
 		)
 		(property "Footprint" "TerminalBlock_Phoenix:TerminalBlock_Phoenix_MKDS-1,5-4-5.08_1x04_P5.08mm_Horizontal"
-			(at 246.38 69.85 0)
+			(at 246.38 72.39 0)
 			(effects
 				(font
@@
 		)
 		(property "Datasheet" "~"
-			(at 246.38 69.85 0)
+			(at 246.38 72.39 0)
 			(effects
 				(font
@@
 		)
 		(property "Description" "Generic screw terminal, single row, 01x04, script generated (kicad-library-utils/schlib/autogen/connector/)"
-			(at 246.38 69.85 0)
+			(at 246.38 72.39 0)
 			(effects
 				(font
